Commit message: Update

File: HarvestingRobot/src/dobot_gazebo/urdf/nova5_robot_panther.xacro (robot description, xacro)
@@ -510,5 +510,5 @@
           <geometry>
               <!-- <box size="${d455_cam_depth} ${d455_cam_width} ${d455_cam_height}"/> -->
-              <mesh filename="package://realsense2_description/meshes/d435.dae" />
+              <mesh filename="package://realsense2_description/meshes/d435.stl" scale="0.001 0.001 0.001"/>
           </geometry>
           <material name="aluminum" />
@@ -532,7 +532,7 @@
     <child link="camera_link" />
   </joint>
-  <!-- xacro:sensor_d455 parent="base_link_gripper" use_nominal_extrinsics="$(arg use_nominal_extrinsics)">
-    <origin xyz="0.065 0 0" rpy="0 -1.57 3.14"/>
-  </xacro:sensor_d435 -->
+  <xacro:sensor_d435 name="camera" topics_ns="camera" parent="base_link_gripper" publish_pointcloud="true">
+    <origin xyz="0 0 0" rpy="0 0 0" />
+  </xacro:sensor_d435>
   <link
     name="finger1_link">

File: realsense2_description/urdf/_d435.urdf.xacro (robot description, xacro)
@@ -31,39 +31,4 @@
     <color rgba="0.5 0.5 0.5 1"/>
     </material>
-    <!-- camera body, with origin at bottom screw mount -->
-    <joint name="${name}_joint" type="fixed">
-      <xacro:insert_block name="origin" />
-      <parent link="${parent}"/>
-      <child link="${name}_bottom_screw_frame" />
-    </joint>
-    <link name="${name}_bottom_screw_frame"/>
-    <joint name="${name}_link_joint" type="fixed">
-      <origin xyz="0 ${d435_cam_depth_py} ${d435_cam_depth_pz}" rpy="0 0 0"/>
-      <parent link="${name}_bottom_screw_frame"/>
-      <child link="${name}_link" />
-    </joint>
-    <link name="${name}_link">
-      <visual>
-      <origin xyz="${d435_cam_mount_from_center_offset} ${-d435_cam_depth_py} 0" rpy="${M_PI/2} 0 ${M_PI/2}"/>
-        <geometry>
-          <!-- <box size="${d435_cam_width} ${d435_cam_height} ${d435_cam_depth}"/> -->
-          <mesh filename="package://realsense2_description/meshes/d435.dae" />
-          <!--<mesh filename="package://realsense2_description/meshes/d435/d435.dae" />-->
-        </geometry>
-        <material name="${name}_aluminum"/>
-      </visual>
-      <collision>
-        <origin xyz="0 ${-d435_cam_depth_py} 0" rpy="0 0 0"/>
-        <geometry>
-        <box size="${d435_cam_depth} ${d435_cam_width} ${d435_cam_height}"/>
-        </geometry>
-      </collision>
-      <inertial>
-        <!-- The following are not reliable values, and should not be used for modeling -->
-        <mass value="0.564" />
-        <origin xyz="0 0 0" />
-        <inertia ixx="0.003881243" ixy="0.0" ixz="0.0" iyy="0.000498940" iyz="0.0" izz="0.003879257" />
-      </inertial>
-    </link>
     <!-- camera depth joints and links -->
     <joint name="${name}_depth_joint" type="fixed">

Commit message: Update

File: HarvestingRobot/src/dobot_gazebo/urdf/nova5_robot_panther.xacro (robot description, xacro)
@@ -3,4 +3,9 @@
   <xacro:include filename="camera.xacro"/>
   <xacro:include filename="$(find realsense2_description)/urdf/_d435.urdf.xacro" />
+  <!--
+  SET CAMERA POSITION AND FOV OFFSET HERE
+  -->
+  <xacro:property name="camera_position" value="0.011150000000000002 0 0.0145"/>
+  <xacro:property name="fov_offset" value="0.00465 0 0"/>
   <link name="world"/>
   <joint
@@ -15,5 +20,5 @@
   <xacro:property name="r" value="0.08" />
   <xacro:property name="h" value="0.20" />
-  <xacro:property name="limit" value="4000000"/>
+  <xacro:property name="limit" value="40000"/>
     <material name="aluminum">
         <color rgba="0.5 0.5 0.5 1" />
@@ -507,5 +512,5 @@
           <!-- the mesh origin is at front plate in between the two infrared camera axes -->
           <!-- <origin xyz="${d455_zero_depth_to_glass-d455_cam_depth/2} ${-d455_cam_depth_py} 0" rpy="0 0 0"/> -->
-          <origin rpy="1.5707963267948966 0 1.5707963267948966" xyz="0.0046500000000000005 -0.0475 0" />
+          <origin rpy="1.5707963267948966 0 1.5707963267948966" xyz="${fov_offset}" />
           <geometry>
               <!-- <box size="${d455_cam_depth} ${d455_cam_width} ${d455_cam_height}"/> -->
@@ -528,5 +533,5 @@
   </link>
   <joint name="camera_link_joint" type="fixed">
-    <origin rpy="0 0 0" xyz="0.011150000000000002 0.0475 0.0145" />
+    <origin rpy="0 0 0" xyz="${camera_position}" />
     <parent link="camera_bottom_screw_frame" />
     <child link="camera_link" />

Commit message: Update

File: HarvestingRobot/src/dobot_gazebo/urdf/nova5_robot_panther.xacro (robot description, xacro)
@@ -12,19 +12,19 @@
     name="world_joint"
     type="fixed">
-    <origin xyz="0 0 0" rpy="0 0 0"/>
+    <origin xyz="0 0 0.16" rpy="0 0 0"/>
     <parent
       link="world" />
     <child
-      link="base_link" />
+      link="mobile_platform_link" />
   </joint>
   <xacro:property name="r" value="0.08" />
   <xacro:property name="h" value="0.20" />
   <xacro:property name="limit" value="40000"/>
-    <material name="aluminum">
-        <color rgba="0.5 0.5 0.5 1" />
-    </material>
-    <material name="plastic">
-        <color rgba="0.1 0.1 0.1 1" />
-    </material>
+  <material name="aluminum">
+      <color rgba="0.5 0.5 0.5 1" />
+  </material>
+  <material name="plastic">
+      <color rgba="0.1 0.1 0.1 1" />
+  </material>
   <!-- <link name="cylinder_link">
     <visual>
@@ -74,4 +74,49 @@
       link="base_link" />
   </joint> -->
+  <link name="mobile_platform_link">
+    <visual>
+      <origin xyz="0 0 0" rpy="0 0 0"/>
+      <geometry>
+         <mesh
+          filename="package://dobot_description/meshes/nova5/panther.stl" scale="0.001 0.001 0.001"/>
+      </geometry>
+    </visual>
+    <inertial>
+      <origin xyz="0 0 0.04" rpy="0 0 0"/>
+      <mass value="0.01"/>
+      <inertia ixx="0.00308109148952278"
+        ixy="-4.0369958400766E-08"
+        ixz="5.2607663395944E-07"
+        iyy="0.00309758743296662"
+        iyz="-6.37484696538659E-09"
+        izz="0.00232835367593981" />
+    </inertial>
+    <collision>
+      <origin xyz="0 0 0" rpy="0 0 0"/>
+      <geometry>
+         <box size="0.1 0.1 0.1"/>
+      </geometry>
+    </collision>
+  </link>
+  <gazebo reference="mobile_platform_link">
+    <material>Gazebo/Grey</material>
+    <dampingFactor>0.05</dampingFactor>
+    <kp>1000000</kp>
+    <kd>1.0</kd>
+    <mu1>100.0</mu1>
+    <mu2>100.0</mu2>
+    <minDepth>0.001</minDepth>
+  </gazebo>
+  <joint
+    name="robot_joint"
+    type="fixed">
+    <origin
+      xyz="0 0 0.13"
+      rpy="0 0 0" />
+    <parent
+      link="mobile_platform_link" />
+    <child
+      link="base_link" />
+  </joint>
   <link
     name="base_link">

Commit message: Update

File: HarvestingRobot/src/dobot_gazebo/urdf/nova5_robot_panther.xacro (robot description, xacro)
@@ -3,9 +3,12 @@
   <xacro:include filename="camera.xacro"/>
   <xacro:include filename="$(find realsense2_description)/urdf/_d435.urdf.xacro" />
-  <!--
-  SET CAMERA POSITION AND FOV OFFSET HERE
-  -->
+  <!-- SET CAMERA POSITION AND FOV OFFSET HERE -->
   <xacro:property name="camera_position" value="0.011150000000000002 0 0.0145"/>
   <xacro:property name="fov_offset" value="0.00465 0 0"/>
+   <xacro:property name="platform_type" value="panther"/>
+   <!-- PLATFORM TYPES
+   panther
+   hunter
+   -->
   <link name="world"/>
   <joint
@@ -79,5 +82,5 @@
       <geometry>
          <mesh
-          filename="package://dobot_description/meshes/nova5/panther.stl" scale="0.001 0.001 0.001"/>
+          filename="package://dobot_description/meshes/nova5/${platform_type}.stl" scale="0.001 0.001 0.001"/>
       </geometry>
     </visual>

File: realsense2_description/urdf/_d435.gazebo.xacro (robot description, xacro)
@@ -1,8 +1,3 @@
 <?xml version="1.0"?>
-<!--
-License: Apache 2.0. See LICENSE file in root directory.
-Copyright(c) 2017 PAL Robotics, S.L. All Rights Reserved
-This is the Gazebo URDF model for the Intel RealSense D435 camera
--->
 <robot xmlns:xacro="http://ros.org/wiki/xacro">
   <xacro:macro name="gazebo_d435" params="camera_name reference_link topics_ns depth_optical_frame color_optical_frame infrared1_optical_frame infrared2_optical_frame publish_pointcloud:=true" >
