Commit message: Update
Make camera mounting position (arm or platform) variabler via .bashrc (CAMERA_POSITION)

File: software_justin/HarvestingRobot/src/dobot_gazebo/urdf/nova5_robot_hunter_camera_on_arm.xacro (robot description, xacro)
@@ -3,6 +3,7 @@
   <xacro:include filename="camera.xacro"/>
   <xacro:include filename="$(find realsense2_description)/urdf/_d435.urdf.xacro" />
-  <!-- SET CAMERA POSITION AND FOV OFFSET HERE -->
+  <!-- SET CAMERA POSE AND FOV OFFSET HERE -->
   <xacro:property name="camera_position" value="0.011150000000000002 0 0.0145"/>
+  <xacro:property name="camera_orientation" value="0 0 0"/>
   <xacro:property name="fov_offset" value="0.00465 0 0"/>
    <xacro:property name="platform_type" value="hunter"/>
@@ -581,5 +582,5 @@
   </link>
   <joint name="camera_link_joint" type="fixed">
-    <origin rpy="0 0 0" xyz="${camera_position}" />
+    <origin rpy="${camera_orientation}" xyz="${camera_position}" />
     <parent link="camera_bottom_screw_frame" />
     <child link="camera_link" />

File: software_justin/HarvestingRobot/src/dobot_gazebo/urdf/nova5_robot_panther_camera_on_arm.xacro (robot description, xacro)
@@ -3,6 +3,7 @@
   <xacro:include filename="camera.xacro"/>
   <xacro:include filename="$(find realsense2_description)/urdf/_d435.urdf.xacro" />
-  <!-- SET CAMERA POSITION AND FOV OFFSET HERE -->
+  <!-- SET CAMERA POSE AND FOV OFFSET HERE -->
   <xacro:property name="camera_position" value="0.011150000000000002 0 0.0145"/>
+  <xacro:property name="camera_orientation" value="0 0 0"/>
   <xacro:property name="fov_offset" value="0.00465 0 0"/>
    <xacro:property name="platform_type" value="panther"/>
@@ -581,5 +582,5 @@
   </link>
   <joint name="camera_link_joint" type="fixed">
-    <origin rpy="0 0 0" xyz="${camera_position}" />
+    <origin rpy="${camera_orientation}" xyz="${camera_position}" />
     <parent link="camera_bottom_screw_frame" />
     <child link="camera_link" />
