Commit message: Update

File: software_justin/HarvestingRobot/src/dobot_gazebo/urdf/nova5_robot_panther_camera_on_platform.xacro (robot description, xacro)
@@ -4,5 +4,7 @@
   <xacro:include filename="$(find realsense2_description)/urdf/_d435.urdf.xacro" />
   <!-- SET CAMERA POSITION AND FOV OFFSET HERE -->
-  <xacro:property name="camera_position" value="0.011150000000000002 0 0.0145"/>
+  <!-- <xacro:property name="camera_position" value="0.011150000000000002 0 0.0145"/> -->
+  <xacro:property name="camera_position" value="0.011150000000000002 0 0"/>
+  <xacro:property name="camera_orientation" value="0 0 0"/>
   <xacro:property name="fov_offset" value="0.00465 0 0"/>
    <xacro:property name="platform_type" value="panther"/>
@@ -115,5 +117,5 @@
     type="fixed">
     <origin
-      xyz="0 0 0.13"
+      xyz="0 0 0.5"
       rpy="0 0 0" />
     <parent
@@ -595,5 +597,5 @@
   </xacro:sensor_d435>   -->
   <joint name="camera_link_joint" type="fixed">
-    <origin rpy="0 0 0" xyz="${camera_position}" />
+    <origin rpy="${camera_orientation}" xyz="${camera_position}" />
     <parent link="camera_bottom_screw_frame" />
     <child link="camera_link" />

File: software_justin/realsense2_description/urdf/_d435.gazebo.xacro (robot description, xacro)
@@ -124,10 +124,10 @@
         <infrared1OpticalframeName>${infrared1_optical_frame}</infrared1OpticalframeName>
         <infrared2OpticalframeName>${infrared2_optical_frame}</infrared2OpticalframeName>
-        <rangeMinDepth>0.2</rangeMinDepth>
-        <rangeMaxDepth>10.0</rangeMaxDepth>
+        <rangeMinDepth>0.01</rangeMinDepth>
+        <rangeMaxDepth>100000.0</rangeMaxDepth>
         <pointCloud>${publish_pointcloud}</pointCloud>
         <pointCloudTopicName>depth/color/points</pointCloudTopicName>
-        <pointCloudCutoff>0.25</pointCloudCutoff>
-        <pointCloudCutoffMax>9.0</pointCloudCutoffMax>
+        <pointCloudCutoff>0.02</pointCloudCutoff>
+        <pointCloudCutoffMax>100001.0</pointCloudCutoffMax>
       </plugin>
     </gazebo>
